File: WaterSensor/MCU.kicad_sch (KiCad schematic)
At the start: 9 parts, among them SW1 SW_Push, U1 STM32G491RET6, U3 SRV05-4

Commit message: schematic done
Parts:
- removed U3: SRV05-4, Package_TO_SOT_SMD:SOT-23-6, symbol Power_Protection:SRV05-4
Connections:
- net VREF+: now reaches U1.28 (VREF+)
- net USART3_TX: now reaches U1.30 (PB10)
- net USART3_RX: now reaches U1.33 (PB11)
- net EN_LIN: now reaches U1.44 (PA10)
- net UART4_TX: now reaches U1.52 (PC10)
- net UART4_RX: now reaches U1.53 (PC11)
- no-connect marks 0 -> 33
Other:
- moved on the sheet: C1, C2, C3, RBOOT, RP1, SW1, XTAL1

Commit message: ready to manufacture
Parts:
- added D8: Blue, LED_SMD:LED_0603_1608Metric, symbol Device:LED_Small
- added R24: 120, Resistor_SMD:R_0603_1608Metric, symbol Device:R_Small
- C1, C2, C3: footprint (none) -> Capacitor_SMD:C_0603_1608Metric
- R25: renamed from RBOOT; footprint (none) -> Resistor_SMD:R_0603_1608Metric
- R26: renamed from RP1; footprint (none) -> Resistor_SMD:R_0603_1608Metric
- SW1: footprint (none) -> Button_Switch_SMD:SW_TS04-66-43-BK-160-SMT
- XTAL1: footprint FA-128_2x1p6_SEC -> FA-128-24.0000MB-W0:FA-128_2x1p6_SEC
Connections:
- net EN_LIN: now also U1.45 (PA11); no longer U1.44 (PA10)
- net GND: now also D8.1 (K); no longer U1.6 (PF1)
- net IN_A: now also U1.21 (PA7); no longer U1.20 (PA6)
- net IN_B: now also U1.20 (PA6); no longer U1.21 (PA7)
- net OSC_OUT: now reaches C3.1, XTAL1.3
- net OSC_OUT: now also U1.6 (PF1)
- net BLKC_SEL_A: now reaches U1.38 (PC6)
- net BLKC_SEL_B: now reaches U1.39 (PC7)
- net BLKC_SEL_C: now reaches U1.40 (PC8)
- net BLKC_CTRL_IN: now reaches U1.41 (PC9)
- net uC_Alive: now reaches U1.46 (PA12)
- net uC_Alive: now also R24.1
- net UART4_RX: no longer names the net of U1.53 (PC11)
- net UART4_TX: no longer names the net of U1.52 (PC10)
- new net: D8.2 (A), R24.2
- no-connect marks 33 -> 30
