File: WaterSensor/WaterSensor.kicad_sch (KiCad schematic)
At the start: 9 parts, among them J1 Conn_02x07_Odd_Even, J2 USB_B_Micro, U13 CH340E

Commit message: schematic done
Parts:
- added C19: 100nF, symbol Device:C_Small
- added C20: 1uF, symbol Device:C_Small
- added C21: 1nF, symbol Device:C_Small
- added D5, D6: SS34, Diode_SMD:D_SMA, symbol Diode:SS34
- added J4: Conn_01x02, symbol Connector_Generic:Conn_01x02
- added JFWA, JFWB, JGWA, JGWB: ~, symbol Connector_Generic:Conn_01x01
- added R13: 1k, symbol Device:R_Small
- added U14: TLIN1029DRQ1, D0008A_N, symbol TLIN1029DRQ1:TLIN1029DRQ1
- added U3: TPD2E001DZDR, DZD4, symbol TPD2E001DZDR:TPD2E001DZDR
Connections:
- net GND: now also C19.2, C20.2, C21.2, J4.2 (Pin_2), U14.5 (GND), U3.1 (GND)
- net VIConverter/Iout_FW: now also JFWB.1 (Pin_1)
- net VIConverter/Iout_GW: now also JGWB.1 (Pin_1)
- net Vdrive: now also U3.4 (VCC)
- net at J2.2 (D-), U13.2 (UD-): now also U3.3 (IO2)
- net at J2.3 (D+), RP2.2, U13.1 (UD+): now also U3.2 (IO1)
- new net: D6.1 (K), R13.1
- new net: C21.1, J4.1 (Pin_1), R13.2, U14.6 (LIN)
- new net: C19.1, C20.1, D5.1 (K), U14.7 (VSUP)
- new net DAC_PROT&SWITCH/FW_DAC_IN_A: JFWA.1 (Pin_1)
- new net DAC_PROT&SWITCH/GW_DAC_IN_A: JGWA.1 (Pin_1)
- new net EN_LIN: U14.2 (EN)
- new net PS_IN: D5.2 (A), D6.2 (A)
- new net USART3_RX: U14.4 (TXD)
- new net USART3_TX: U14.1 (RXD)
- no-connect marks 10 -> 12
Other:
- sheet DAC_PROT&SWITCH ports: added FW_DAC_IN_A, FW_DAC_IN_B, GW_DAC_IN_A, GW_DAC_IN_B; removed DAC_A_IN_FW, DAC_A_IN_GW, DAC_B_IN_FW, DAC_B_IN_GW
- sheet MCU ports: added EN_LIN, USART3_RX, USART3_TX, VREF+; removed none
- sheet VIConverter ports: added FW_DAC_IN_B, GW_DAC_IN_B; removed DAC_A_IN_FW, DAC_A_IN_GW
- note added: "DAC-ADAPTER"
- note added: "DAC2CURRENT-CONV"
- note added: "LIN-UART"
- note added: "MCU"
- note added: "POWER SUPPLY"
- note added: "ST-LINK"
- note added: "USB-UART"
- moved on the sheet: C9, D2, D3, D4, J1, J2, R5, RP2, U13

Commit message: ready to manufacture
Parts:
- removed D2, D5, D6: SS34, Diode_SMD:D_SMA, symbol Diode:SS34
- removed J2: USB_B_Micro, symbol Connector:USB_B_Micro
- removed JFWA, JFWB, JGWA, JGWB: ~, symbol Connector_Generic:Conn_01x01
- added D2, D3, D4: 1N5819WS, Diode_SMD:D_SOD-323, symbol Diode:1N5819WS
- added FID1, FID2, FID3: Fiducial, Fiducial:Fiducial_1mm_Mask2mm, symbol Mechanical:Fiducial
- added H1, H2: MountingHole, MountingHole:MountingHole_2.2mm_M2, symbol Mechanical:MountingHole
- added J4: BLK8C, Connector_Molex:Conn_1x5_MicroFit_436500527, symbol Connector_Generic:Conn_01x05
- added J5: BLK9C, Connector_Molex:Conn_1x4_MicroFit_0436500427, symbol Connector_Generic:Conn_01x04
- added J6: USB_B_Mini, Connector_USB:USB_Mini-B_Wuerth_65100516121_Horizontal, symbol Connector:USB_B_Mini
- added J7: BLKA, Connector_Molex:Conn_1x3_MicroFit_436500327, symbol Connector_Generic:Conn_01x03
- added J8: BLKB, Connector_Molex:Conn_1x3_MicroFit_436500327, symbol Connector_Generic:Conn_01x03
- added R17, R18, R19: 22, Resistor_SMD:R_0603_1608Metric, symbol Device:R_Small
- added R22: 220, Resistor_SMD:R_0603_1608Metric, symbol Device:R_Small
- added R23: 120, Resistor_SMD:R_0603_1608Metric, symbol Device:R_Small
- C19, C20, C21, C9: footprint (none) -> Capacitor_SMD:C_0603_1608Metric
- D5: renamed from D4; value LED -> Yellow; footprint (none) -> LED_SMD:LED_0603_1608Metric
- D6: renamed from D3; value LED -> Green; footprint (none) -> LED_SMD:LED_0603_1608Metric
- J1: value Conn_02x07_Odd_Even -> ST-LINK; footprint (none) -> Connector_IDC:Connector_IDC_02x07_1_27mm_SMD
- J3: renamed from J4; value Conn_01x02 -> LIN; footprint (none) -> Connector_Molex:Conn_1x2_MiniFit_1724480002
- R11: renamed from R13; footprint (none) -> Resistor_SMD:R_0603_1608Metric
- R20: renamed from R5; footprint (none) -> Resistor_SMD:R_0603_1608Metric
- R27: renamed from RP2; footprint (none) -> Resistor_SMD:R_0603_1608Metric
- U12: renamed from U14; footprint D0008A_N -> TLIN1029DRQ1:D0008A_N
- U7: renamed from U3; value TPD2E001DZDR -> TPD2E001DRLR; footprint DZD4 -> TPD2E001DRLR:DRL5-M
- renumbered U13 to U10
Connections:
- net +3.3V: now also R22.1, R23.1; no longer D5.2 (A), D6.2 (A)
- net DAC_PROT&SWITCH/FW_DAC_IN_A: now also J7.3 (Pin_3)
- net DAC_PROT&SWITCH/GW_DAC_IN_A: now also J7.2 (Pin_2)
- net GND: now also J6.5 (GND)
- net NRST: now also R19.2; no longer J1.12 (Pin_12)
- net SWCLK: now also R18.2; no longer J1.6 (Pin_6)
- net SWDIO: now also R17.2; no longer J1.4 (Pin_4)
- net USART2_RX: now also U12.4 (TXD); no longer D6.1 (K), U10.8 (TXD)
- net USART2_TX: now also U12.1 (RXD); no longer D5.1 (K), U10.9 (RXD)
- net USART3_RX: now also D6.1 (K), U10.8 (TXD); no longer U12.4 (TXD)
- net USART3_TX: now also D5.1 (K), U10.9 (RXD); no longer U12.1 (RXD)
- net VIConverter/Iout_FW: now also J8.3 (Pin_3)
- net VIConverter/Iout_GW: now also J8.2 (Pin_2)
- net Vdrive: now also D2.1 (K); no longer U7.4 (VCC)
- net at R11.1: now also D4.1 (K)
- net LIN_BUS: now reaches C21.1, J3.1 (Pin_1), R11.2, U12.6 (LIN)
- net USB_D+: now reaches R27.2, U10.1 (UD+), U7.2 (IO1)
- net USB_D+: now also J6.3 (D+)
- net USB_D-: now reaches U10.2 (UD-), U7.3 (IO2)
- net USB_D-: now also J6.2 (D-)
- net at C19.1, C20.1, U12.7 (VSUP): now also D3.1 (K)
- new net: J1.4 (Pin_4), R17.1
- new net: J1.12 (Pin_12), R19.1
- new net: D6.2 (A), R23.2
- new net: D2.2 (A), J6.1 (VBUS)
- new net: D5.2 (A), R22.2
- new net: J1.6 (Pin_6), R18.1
- new net +5V: U7.4 (VCC)
- new net BLK-C-Water/BLK8C-2: J4.2 (Pin_2)
- new net BLK-C-Water/BLK8C-3: J4.3 (Pin_3)
- new net BLK-C-Water/BLK8C-4: J4.4 (Pin_4)
- new net BLK-C-Water/BLK8C-5: J4.5 (Pin_5)
- new net BLK-C-Water/BLK9C-2: J5.1 (Pin_1)
- new net BLK-C-Water/BLK9C-3: J5.2 (Pin_2)
- new net BLK-C-Water/BLK9C-4: J5.3 (Pin_3)
- new net BLK-C-Water/BLK9C-5: J5.4 (Pin_4)
- new net BLK-C-Water/BLKC_PWR: J4.1 (Pin_1)
- new net DAC_PROT&SWITCH/BLKA_PWR: J7.1 (Pin_1)
- new net DAC_PROT&SWITCH/BLKB_PWR: J8.1 (Pin_1)
- new net PS_RAW: D3.2 (A), D4.2 (A)
Other:
- added sheet BLK-C-Water (blk_c_water.kicad_sch)
- sheet DAC_PROT&SWITCH ports: added BLKA_PWR, BLKB_PWR; removed none
- sheet MCU ports: added BLKC_CTRL_IN, BLKC_SEL_A, BLKC_SEL_B, BLKC_SEL_C; removed none
- note added: "BLKC-WATER-CTRL"
- note added: "DAC-CONTROLLED-CURRENT-PUMP"
- note added: "LIN Connector"
- note removed: "DAC2CURRENT-CONV"
- moved on the sheet: C9, D5, D6, U7
