File: WaterSensor/dac_prot&switch.kicad_sch (KiCad schematic)
At the start: 9 parts, among them U10 ${SIM.PARAMS}, U6 TS5A23157QDGSRQ1, U7 ${SIM.PARAMS}, U8 ${SIM.PARAMS}, U9 ${SIM.PARAMS}

Commit message: schematic done
Connections:
- net DAC_A_IN_FW renamed FW_DAC_IN_A
- net DAC_A_IN_GW renamed GW_DAC_IN_A
- net DAC_B_IN_FW renamed FW_DAC_IN_B
- net DAC_B_IN_GW renamed GW_DAC_IN_B
Other:
- note added: "With a LOW Input(IN1 or IN2), NC channel is connected to COM by default"
- note removed: "With a LOW Input, NC channel is connected to COM by default"
Changed lines of the file:
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@@
 		)
 	)
-	(text "With a LOW Input, NC channel is connected to COM by default\n"
+	(text "With a LOW Input(IN1 or IN2), NC channel is connected to COM by default\n"
 		(exclude_from_sim no)
 		(at 122.174 40.132 0)
@@
 		)
 	)
-	(hierarchical_label "DAC_B_IN_FW"
+	(hierarchical_label "FW_DAC_IN_B"
 		(shape output)
 		(at 208.28 97.79 0)
@@
 		)
 	)
-	(hierarchical_label "DAC_B_IN_GW"
+	(hierarchical_label "GW_DAC_IN_B"
 		(shape output)
 		(at 170.18 97.79 0)
@@
 		)
 	)
-	(hierarchical_label "DAC_A_IN_FW"
+	(hierarchical_label "FW_DAC_IN_A"
 		(shape output)
 		(at 170.18 74.93 0)
@@
 		)
 	)
-	(hierarchical_label "DAC_A_IN_GW"
+	(hierarchical_label "GW_DAC_IN_A"
 		(shape output)
 		(at 208.28 74.93 0)

Commit message: ready to manufacture
Parts:
- removed U10, U7, U8, U9: ${SIM.PARAMS}, symbol Simulation_SPICE:OPAMP
- added C24, C25, C26, C30, C31, C33: 0.1uF, Capacitor_SMD:C_0603_1608Metric, symbol Device:C_Small
- added TP1: TP1, TestPoint:TestPoint_Pad_D1.5mm, symbol Connector:TestPoint_Small
- added TP2: TP2, TestPoint:TestPoint_Pad_D1.5mm, symbol Connector:TestPoint_Small
- added U14, U2, U3: OPA2990IDR, OPA2990IDR:D8_TEX-M, symbol TSV632:TSV632
- C18, C8: footprint (none) -> Capacitor_SMD:C_0603_1608Metric
- R10: renamed from R8; footprint (none) -> Resistor_SMD:R_0603_1608Metric
- R9: footprint (none) -> Resistor_SMD:R_0603_1608Metric
- U6: footprint DGS0010A_N -> TS5A23157QDGSRQ1:DGS0010A_N
Connections:
- net FW_DAC_IN_A: now also U2.1 (Out1), U2.2 (In1-)
- net FW_DAC_IN_B: now also U3.1 (Out1), U3.2 (In1-)
- net GND: now also C24.2, C25.2, C26.2, C30.2, C31.2, C33.2, U14.4 (VCC-), U2.4 (VCC-), U3.4 (VCC-)
- net GW_DAC_IN_A: now also U2.6 (In2-), U2.7 (Out2)
- net GW_DAC_IN_B: now also U3.6 (In2-), U3.7 (Out2)
- net DAC_B_IN1+: now reaches U6.7 (NC2)
- net DAC_B_IN1+: now also U3.3 (In1+)
- net DAC_A_RAW_F: now reaches C8.2, R10.2, U6.10 (COM1)
- net DAC_B_RAW_F: now reaches C18.1, R9.2, U6.6 (COM2)
- net DAC_A_IN1+: now reaches U6.9 (NC1)
- net DAC_A_IN1+: now also U2.3 (In1+)
- net DAC_B_IN2+: now reaches U6.4 (NO2)
- net DAC_B_IN2+: now also U3.5 (In2+)
- net DAC_A_IN2+: now reaches U6.2 (NO1)
- net DAC_A_IN2+: now also U2.5 (In2+)
- net Vdrive renamed +5V
- net +5V: now also C24.1
- new net BLKA_PWR: C30.1, U14.3 (In1+)
- new net BLKA_PWR_BUFF: C33.1, TP1.1, U14.1 (Out1), U14.2 (In1-), U2.8 (VCC+)
- new net BLKB_PWR: C31.1, U14.5 (In2+)
- new net BLKB_PWR_BUFF: C25.1, TP2.1, U14.6 (In2-), U14.7 (Out2), U3.8 (VCC+)
- new net PS_RAW: C26.1, U14.8 (VCC+)
Other:
- note added: "<== Should have +12V here to insure the RVCORE BLKB is feeding properly"
- note added: "<== Should have +5V here to insure the RVCORE BLKA is feeding properly"
- note added: "ANALOG SW"
- note added: "BLKA"
- note added: "BLKB"
- note added: "Bypass filters for the AN. SW."
- note added: "These DUAL OPAMPS CHIPS are acting as Buffers"
- moved on the sheet: C18, C8, R10, R9, U6
