File: WaterSensor/powerSuplly.kicad_sch (KiCad schematic)
At the start: 20 parts, among them J3 Conn_01x02, U4 LM1117MP-3.3, U5 LM7805MPX/NOPB

Commit message: schematic done
Parts:
- added C22, C23: 2.2uF, symbol Device:C_Small
- added R14: 50, symbol Device:R_Small
- added U15: MCP1501T-33E/CHY, SOT-23-6_CHY_MCH, symbol MCP1501T-33E-CHY:MCP1501T-33E_CHY
Connections:
- net +3.3V: now also C22.1, U15.4 (*SHDN), U15.6 (VDD)
- net GND: now also C22.2, C23.2, U15.2 (GND), U15.3 (GND), U15.5 (GND)
- new net: C23.1, R14.2
- new net VREF+: R14.1, U15.1 (OUT)

Commit message: ready to manufacture
Parts:
- removed D1: SS34, Diode_SMD:D_SMA, symbol Diode:SS34
- added C34: 10uF, Capacitor_SMD:C_0805_2012Metric, symbol Device:C_Small
- added C35: 100nF, Capacitor_SMD:C_0603_1608Metric, symbol Device:C_Small
- added D1: 1N5819WS, Diode_SMD:D_SOD-323, symbol Diode:1N5819WS
- added FB3: HI1206N101R-10, Inductor_SMD:L_0603_1608Metric, symbol Device:FerriteBead_Small
- C10, C11, C12, C13, C14, C16, C17, C22, C23, C4: footprint (none) -> Capacitor_SMD:C_0603_1608Metric
- C15, C5, C6, C7: footprint (none) -> Capacitor_SMD:C_0805_2012Metric
- D7: renamed from PW_LED; value LED -> Red; footprint (none) -> LED_SMD:LED_0603_1608Metric
- FB1: value 100Ohm @ 100Mhz -> HI1206N101R-10; footprint (none) -> Inductor_SMD:L_0603_1608Metric
- FB2: renamed from L2; value 600R -> HZ0603C601R-10; footprint (none) -> Inductor_SMD:L_0603_1608Metric
- J2: renamed from J3; value Conn_01x02 -> PS_IN; footprint (none) -> Connector_Molex:Conn_1x2_MiniFit_1724480002
- R12: renamed from R14; footprint (none) -> Resistor_SMD:R_0603_1608Metric
- R21: renamed from R6; value 3k -> 220; footprint (none) -> Resistor_SMD:R_0603_1608Metric
- U11: renamed from U15; footprint SOT-23-6_CHY_MCH -> MCP1501T-33E-CHY:SOT-23-6_CHY_MCH
- U4: footprint Package_TO_SOT_SMD:SOT-223-3_TabPin2 -> LM1117MPX-33NOPB:SOT223-318H_OSI-M
- U5: footprint DCY4_TEX -> LM7805MPX_NOPB:LM7805MPX_NOPB
Connections:
- net GND: now also C34.2, C35.2
- net PS_IN: now also D1.2 (A)
- net PS_RAW: now reaches C4.1, U5.1 (INPUT)
- net PS_RAW: now also C34.1, C35.1, FB3.2
- net +5V: now reaches C5.1, C6.1, FB1.2, U4.3 (VI), U5.3 (OUTPUT)
- new net: D1.1 (K), FB3.1
Other:
- note added: "Power Connector"
- moved on the sheet: J2
